Commit message: wip

File: urdf/udacity_bot.xacro (robot description, xacro)
@@ -138,5 +138,5 @@
     <joint_properties damping="1.0" friction="1.0"/>
   </joint>
-  <link name='camera'>
+  <link name='camera_link'>
     <inertial>
       <mass value="0.1"/>
@@ -163,5 +163,5 @@
   <joint type="fixed" name="camera_joint">
     <origin xyz="0.2 0  0" rpy="0 0 0"/>
-    <child link="camera"/>
+    <child link="camera_link"/>
     <parent link="chassis"/>
     <axis xyz="0 1 0" rpy="0 0 0"/>
